File: NRF52832-base/NRF52832 Lipo/NRF52832 Base.kicad_pcb (KiCad board)
At the start: 2 copper layers, 38.7 x 19 mm, 39 parts, among them J1 Conn_01x06, J2 USB_B_Micro, Q1 CJ3139K, U1 NRF52832-QFAA-R, U3 AP2112K-3.3, U4 TP4054ST, U5 CP2104, Y1 32MHz, Y2 32.768kHz

Commit message: updating pdfs
Parts:
- J1: footprint Connector_PinSocket_1.00mm:PinSocket_2x02_P1.00mm_Vertical_SMD -> Connector_PinHeader_1.27mm:PinHeader_2x02_P1.27mm_Vertical_SMD
- Q1: footprint Package_TO_SOT_SMD:SOT-723 -> Package_DFN_QFN:Diodes_DFN1006-3
- U2: value (none) -> ProMicro
- moved J1 2.01 mm to (139.6, 94.1), turned to 180 degrees
Connections:
- J1 pad 1: VCC -> SWDIO
- J1 pad 2: GND -> SWDCLK
- J1 pad 3: SWDIO -> VCC
- J1 pad 4: SWDCLK -> GND
Routing:
- net VCC: track 46.8 -> 54.6 mm, vias 4 -> 5
- net SWDIO: track 4.87 -> 7.39 mm
- net SWDCLK: track 1.48 -> 3.75 mm
- net GND: track 141.7 -> 142.2 mm, vias 27 -> 26
- net Net-(C6-Pad1): vias 0 -> 2
Other:
- board text added: "BlueNano V2.0.1"
- board text removed: "BlueNano V2.0"

Commit message: bringing all changes and tests in here
Parts:
- Q1: value CJ3139K -> LP0404N3T5G
Changed lines of the file:
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@@
       (effects (font (size 1 1) (thickness 0.15)))
     )
-    (fp_text value CJ3139K (at 0 1.6 270) (layer F.Fab)
+    (fp_text value LP0404N3T5G (at 0 1.6 270) (layer F.Fab)
       (effects (font (size 1 1) (thickness 0.15)))
     )
@@
   (via (at 127.508 92.329) (size 0.6) (drill 0.3) (layers F.Cu B.Cu) (net 2))
   (via (at 125.73 85.852) (size 0.6) (drill 0.3) (layers F.Cu B.Cu) (net 2))
-  (via (at 134.493 94.869) (size 0.6) (drill 0.3) (layers F.Cu B.Cu) (net 6))
   (via (at 143.002 98.298) (size 0.6) (drill 0.3) (layers F.Cu B.Cu) (net 2))
   (via (at 143.002 97.409) (size 0.6) (drill 0.3) (layers F.Cu B.Cu) (net 2))
@@
   (segment (start 130.77441 84.87661) (end 130.509168 84.611368) (width 0.1524) (layer F.Cu) (net 5))
   (segment (start 132.43788 84.87661) (end 130.77441 84.87661) (width 0.1524) (layer F.Cu) (net 5))
+  (via (at 134.493 94.869) (size 0.6) (drill 0.3) (layers F.Cu B.Cu) (net 6))
   (segment (start 129.396477 90.770832) (end 129.396477 90.770832) (width 0.254) (layer F.Cu) (net 6))
   (via (at 133.731 84.582) (size 0.6) (drill 0.3) (layers F.Cu B.Cu) (net 6))
