File: NRF52832-base/NRF52832 Lipo/NRF52832 Base.sch (KiCad schematic (older format))
At the start: 39 parts, among them J1 Conn_01x06, J2 USB_B_Micro, Q1 CJ3139K, U1 NRF52832-QFAA-R, U2 ProMicro, U3 AP2112K-3.3, U4 TP4054ST, U5 CP2104, Y1 32MHz, Y2 32.768kHz

Commit message: updating pdfs
Parts:
- J1: footprint Connector_PinSocket_1.00mm:PinSocket_2x02_P1.00mm_Vertical_SMD -> Connector_PinHeader_1.27mm:PinHeader_2x02_P1.27mm_Vertical_SMD
- Q1: footprint Package_TO_SOT_SMD:SOT-723 -> Package_DFN_QFN:Diodes_DFN1006-3
Changed lines of the file:
@@
 F 0 "J1" H 5570 925 50  0000 C CNN
 F 1 "Conn_01x06" H 5570 1016 50  0000 C CNN
-F 2 "Connector_PinSocket_1.00mm:PinSocket_2x02_P1.00mm_Vertical_SMD" H 5650 1450 50  0001 C CNN
+F 2 "Connector_PinHeader_1.27mm:PinHeader_2x02_P1.27mm_Vertical_SMD" H 5650 1450 50  0001 C CNN
 F 3 "~" H 5650 1450 50  0001 C CNN
 	1    5650 1450
@@
 Wire Wire Line
 	6050 1550 5850 1550
-Text GLabel 5950 1250 2    50   Input ~ 0
+Text GLabel 6050 1450 2    50   Input ~ 0
 SWDCLK
-Text GLabel 6050 1350 2    50   Input ~ 0
+Text GLabel 6050 1550 2    50   Input ~ 0
 SWDIO
 $Comp
 L power:GND #PWR014
 U 1 1 5BB7854F
-P 6050 1450
-F 0 "#PWR014" H 6050 1200 50  0001 C CNN
-F 1 "GND" V 6055 1322 50  0000 R CNN
-F 2 "" H 6050 1450 50  0001 C CNN
-F 3 "" H 6050 1450 50  0001 C CNN
-	1    6050 1450
+P 5950 1250
+F 0 "#PWR014" H 5950 1000 50  0001 C CNN
+F 1 "GND" V 5955 1122 50  0000 R CNN
+F 2 "" H 5950 1250 50  0001 C CNN
+F 3 "" H 5950 1250 50  0001 C CNN
+	1    5950 1250
 	0    -1   -1   0
 $EndComp
@@
 L power:VCC #PWR015
 U 1 1 5BB7869C
-P 6050 1550
-F 0 "#PWR015" H 6050 1400 50  0001 C CNN
-F 1 "VCC" V 6067 1678 50  0000 L CNN
-F 2 "" H 6050 1550 50  0001 C CNN
-F 3 "" H 6050 1550 50  0001 C CNN
-	1    6050 1550
+P 6050 1350
+F 0 "#PWR015" H 6050 1200 50  0001 C CNN
+F 1 "VCC" V 6067 1478 50  0000 L CNN
+F 2 "" H 6050 1350 50  0001 C CNN
+F 3 "" H 6050 1350 50  0001 C CNN
+	1    6050 1350
 	0    1    1    0
 $EndComp
@@
 F 0 "Q1" H 4656 6896 50  0000 L CNN
 F 1 "CJ3139K" H 4656 6805 50  0000 L CNN
-F 2 "Package_TO_SOT_SMD:SOT-723" H 4650 6775 50  0001 L CIN
+F 2 "Package_DFN_QFN:Diodes_DFN1006-3" H 4650 6775 50  0001 L CIN
 F 3 "https://lcsc.com/product-detail/MOSFET_P5102FM_C133604.html" H 4450 6850 50  0001 L CNN
 	1    4450 6850

Commit message: bringing all changes and tests in here
Parts:
- Q1: value CJ3139K -> LP0404N3T5G
Changed lines of the file:
@@
 P 4450 6850
 F 0 "Q1" H 4656 6896 50  0000 L CNN
-F 1 "CJ3139K" H 4656 6805 50  0000 L CNN
+F 1 "LP0404N3T5G" H 4656 6805 50  0000 L CNN
 F 2 "Package_DFN_QFN:Diodes_DFN1006-3" H 4650 6775 50  0001 L CIN
 F 3 "https://lcsc.com/product-detail/MOSFET_P5102FM_C133604.html" H 4450 6850 50  0001 L CNN
