File: 4x4_backpack_nrf52840/4x4_backpack.kicad_pcb (KiCad board)
At the start: 2 copper layers, 76.2 x 76.2 mm, 44 parts, among them J1 Conn_01x04, J10 TC2050, J11 Conn_01x01, J12 Conn_01x01, J13 Conn_01x01, J14 Conn_01x01, J15 Conn_01x01, J16 Conn_01x01, J17 USB_B_Micro, J2 Conn_01x04, J3 Conn_01x04, J4 Conn_01x04, J5 Conn_01x04, J6 Conn_01x04, J7 Conn_01x04, J8 Conn_01x04, J9 Conn_01x04, Q1 P5102FM, SW1 SW_SPDT, SW2 RESET, U1 E73-2G4M08S1C, U2 TP4056, U3 AP2112K-3.3, Y1 32.768kHz

Commit message: adding 840backpack
Parts:
- added D4: LED, LED_SMD:LED_0805_2012Metric_Pad1.15x1.40mm_HandSolder, F.Cu at (92.5, 134.0)
- added D5: LED, LED_SMD:LED_0805_2012Metric_Pad1.15x1.40mm_HandSolder, F.Cu at (98.8, 134.0)
- added L1: DNP, Inductor_SMD:L_0805_2012Metric_Pad1.15x1.40mm_HandSolder, F.Cu at (108.5, 101.5)
- added R10: 1k, Resistor_SMD:R_0805_2012Metric_Pad1.15x1.40mm_HandSolder, F.Cu at (98.8, 129.2)
- added R9: 1k, Resistor_SMD:R_0805_2012Metric_Pad1.15x1.40mm_HandSolder, F.Cu at (92.5, 129.5)
- C17, C18: value 12pF -> 22pF
Connections:
- D3 pad 4: /P1.02 -> WS2812
- U1 pad 10: COL4 -> COL3
- U1 pad 12: (no net) -> COL4
- U1 pad 14: (no net) -> COL5
- U1 pad 15: COL5 -> COL6
- U1 pad 16: (no net) -> COL7
- U1 pad 17: COL6 -> COL8
- U1 pad 2: ROW2 -> BLUE_LED
- U1 pad 24: (no net) -> GND
- U1 pad 25: (no net) -> Net-(L1-Pad1)
- U1 pad 28: COL12 -> WS2812
- U1 pad 3: ROW3 -> ROW2
- U1 pad 30: COL11 -> COL12
- U1 pad 32: COL10 -> COL11
- U1 pad 33: COL7 -> COL10
- U1 pad 35: COL8 -> COL16
- U1 pad 38: /P1.02 -> (no net)
- U1 pad 4: ROW4 -> ROW3
- U1 pad 40: COL16 -> RED_LED
- U1 pad 6: COL1 -> ROW4
- U1 pad 7: COL2 -> COL1
- U1 pad 8: COL3 -> COL2
Routing:
- net WS2812: track 0.00 -> 96.7 mm, vias 0 -> 2
- net /P1.02: track 96.4 -> 0.00 mm, vias 1 -> 0
- net BLUE_LED: track 0.00 -> 63.2 mm, vias 0 -> 4
- net RED_LED: track 0.00 -> 55.3 mm, vias 0 -> 1
- net GND: track 157.2 -> 166.6 mm, vias 87 -> 101
- net COL8: track 122.0 -> 113.1 mm
- net COL7: track 117.5 -> 110.6 mm, vias 3 -> 2
- net COL10: track 145.5 -> 151.8 mm, vias 2 -> 3
- net Net-(D5-Pad1): track 0.00 -> 5.60 mm
- net Net-(D4-Pad1): track 0.00 -> 5.32 mm
- net Net-(L1-Pad1): track 0.00 -> 4.19 mm
- net COL16: track 82.7 -> 79.5 mm, vias 1 -> 2
- net COL4: track 22.7 -> 25.5 mm
- net RESET: track 64.5 -> 66.6 mm
- net COL5: track 105.1 -> 106.4 mm, vias 1 -> 0
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