File: BlueMicro2.0a/EByte_E73.kicad_pcb (KiCad board)
At the start: 2 copper layers, 21.6 x 62.2 mm, 25 parts, among them J1 USB_OTG, J2 Serial Connector, J3 Conn_01x02, Q1 DMG3415U, U1 E73-2G4M04S, U2 ProMicro, U3 AP2112K-3.3, U6 TP4056

Commit message: adding 840backpack
Parts:
- removed JP3: JUMPER-SMT_2_NO, E73:SolderJumperSingle
- added C9: 0.1uF, Capacitors_SMD:C_0805_HandSoldering, F.Cu at (106.3, 142.4)
- added JP1: JUMPER-SMT_2_NO, E73:SolderJumperSingle, F.Cu at (103.5, 148.3)
- added R6: 1K, Resistors_SMD:R_0805_HandSoldering, F.Cu at (106.3, 144.4)
- added U4: CH340C, SMD_Packages:SO-16-N, B.Cu at (109.2, 143.7)
- U3, U6: moved to B.Cu
- moved C5 8.28 mm to (114.4, 137.3)
- moved C7 8.03 mm to (111.0, 134.2), turned to 0 degrees
- moved Q1 7.75 mm to (111.0, 137.2), turned to 180 degrees
- moved R2 6.30 mm to (112.2, 142.3), turned to 0 degrees
- moved C8 6.23 mm to (112.3, 144.4), turned to 0 degrees
- moved D1 3.64 mm to (106.2, 139.4)
- moved U6 2.04 mm to (110.5, 135.4)
- moved R3 0.46 mm to (111.0, 132.3), turned to 0 degrees
- moved U3 0.10 mm to (105.4, 129.8)
Connections:
- J1 pad 2: (no net) -> /Data-
- J1 pad 3: (no net) -> /Data+
- U2 pad 1: Net-(JP3-Pad2) -> (no net)
Routing:
- net TXD: track 12.8 -> 50.8 mm, vias 0 -> 3
- net RXD: track 12.5 -> 40.0 mm
- net /VBatt: track 69.5 -> 48.5 mm
- net GND: track 187.5 -> 198.8 mm, vias 13 -> 18
- net /VBus: track 30.8 -> 42.1 mm, vias 0 -> 3
- net Net-(C9-Pad1): track 0.00 -> 6.60 mm, vias 0 -> 1
- net Net-(R6-Pad2): track 0.00 -> 5.94 mm, vias 0 -> 1
- net Net-(R3-Pad1): track 2.10 -> 6.70 mm, vias 0 -> 1
- net /DTR: track 0.00 -> 3.73 mm, vias 0 -> 1
- net /Data-: track 0.00 -> 3.19 mm, vias 0 -> 1
- net /Data+: track 0.00 -> 3.00 mm, vias 0 -> 1
- net Net-(JP3-Pad2): track 2.17 -> 0.00 mm
- net RESET: track 70.8 -> 72.3 mm
- net VCC: track 56.3 -> 57.6 mm, vias 2 -> 1
- net Net-(C5-Pad1): track 25.9 -> 25.2 mm, vias 2 -> 1
Other:
- board text added: "For Assembly Instructions, refer to: https://github.com/jpconstantineau /NRF52-Board For Firmware, refer to: https://github.com/jpconstantineau /BlueMicro_BLE"
- board text added: "Jump for DTR Reset"
- board text added: "V2.0"
- board text removed: "Assembly Instructions: https://github.com /jpconstantineau /NRF52-Board Firmware: https://github.com /jpconstantineau /BlueMicro_BLE"
- board text removed: "V2.0b"
