File: TC2050_adapter/TC2050_adapter/TC2050_adapter.sch (KiCad schematic (older format))
At the start: 22 parts, among them J1 Conn_01x05, J10 Conn_01x01, J11 TC2050_pogo, J12 Conn_01x01, J13 Conn_01x01, J14 Conn_01x01, J15 Conn_01x01, J16 Conn_01x01, J17 Conn_01x01, J18 Conn_01x01, J19 Conn_01x01, J2 Cortex Debug 10-pin connector, J20 Conn_01x01, J21 Conn_01x01, J22 Conn_01x01, J3 Conn_01x05, J4 Conn_01x05, J5 TC2050_pogo, J6 Conn_01x05, J7 TC2050_pogo_alignment, J8 TC2050_pogo, J9 TC2050_pogo

Commit message: adding testing jigs
Parts:
- removed J10, J12, J13, J14, J15, J16, J17, J18, J19, J20, J21, J22: Conn_01x01, E73:mouse-bite-2mm-slot, symbol Connector_Generic:Conn_01x01
- removed J5: TC2050_pogo, E73:TC2050_pogo, symbol Connector_Generic:Conn_02x05_Counter_Clockwise
- added J5: Cortex Debug 10-pin connector, Connector_PinHeader_1.27mm:PinHeader_2x05_P1.27mm_Vertical, symbol Connector_Generic:Conn_02x05_Odd_Even
- J11, J8, J9: footprint E73:TC2050_pogo -> Connector_PinSocket_1.27mm:PinSocket_2x05_P1.27mm_Vertical
- J7: footprint E73:TC2050_alignment -> Connector_PinSocket_1.27mm:PinSocket_2x05_P1.27mm_Vertical
Connections:
- no-connect marks 52 -> 40
Changed lines of the file:
@@
 EESchema Schematic File Version 4
+LIBS:TC2050_adapter-cache
 EELAYER 26 0
 EELAYER END
@@
 $EndDescr
 $Comp
-L Connector_Generic:Conn_02x05_Counter_Clockwise J5
-U 1 1 5C9E804A
-P 8800 1550
-F 0 "J5" H 8850 1967 50  0000 C CNN
-F 1 "TC2050_pogo" H 8850 1876 50  0000 C CNN
-F 2 "E73:TC2050_pogo" H 8800 1550 50  0001 C CNN
-F 3 "~" H 8800 1550 50  0001 C CNN
-	1    8800 1550
-	1    0    0    -1
-$EndComp
-$Comp
 L Connector_Generic:Conn_02x05_Odd_Even J2
 U 1 1 5C9E812B
@@
 F 0 "J7" H 8850 3017 50  0000 C CNN
 F 1 "TC2050_pogo_alignment" H 8850 2926 50  0000 C CNN
-F 2 "E73:TC2050_alignment" H 8800 2600 50  0001 C CNN
+F 2 "Connector_PinSocket_1.27mm:PinSocket_2x05_P1.27mm_Vertical" H 8800 2600 50  0001 C CNN
 F 3 "~" H 8800 2600 50  0001 C CNN
 	1    8800 2600
@@
 F 0 "J8" H 8850 3817 50  0000 C CNN
 F 1 "TC2050_pogo" H 8850 3726 50  0000 C CNN
-F 2 "E73:TC2050_pogo" H 8800 3400 50  0001 C CNN
+F 2 "Connector_PinSocket_1.27mm:PinSocket_2x05_P1.27mm_Vertical" H 8800 3400 50  0001 C CNN
 F 3 "~" H 8800 3400 50  0001 C CNN
 	1    8800 3400
@@
 F 0 "J9" H 7850 3817 50  0000 C CNN
 F 1 "TC2050_pogo" H 7850 3726 50  0000 C CNN
-F 2 "E73:TC2050_pogo" H 7800 3400 50  0001 C CNN
+F 2 "Connector_PinSocket_1.27mm:PinSocket_2x05_P1.27mm_Vertical" H 7800 3400 50  0001 C CNN
 F 3 "~" H 7800 3400 50  0001 C CNN
 	1    7800 3400
@@
 NoConn ~ 7600 3500
 $Comp
-L Connector_Generic:Conn_01x01 J10
-U 1 1 5C9F542F
-P 1450 2650
-F 0 "J10" H 1530 2692 50  0000 L CNN
-F 1 "Conn_01x01" H 1530 2601 50  0000 L CNN
-F 2 "E73:mouse-bite-2mm-slot" H 1450 2650 50  0001 C CNN
-F 3 "~" H 1450 2650 50  0001 C CNN
-	1    1450 2650
-	1    0    0    -1
-$EndComp
-NoConn ~ 1250 2650
-$Comp
 L Connector_Generic:Conn_02x05_Counter_Clockwise J11
 U 1 1 5C9F59C3
@@
 F 0 "J11" H 9750 3817 50  0000 C CNN
 F 1 "TC2050_pogo" H 9750 3726 50  0000 C CNN
-F 2 "E73:TC2050_pogo" H 9700 3400 50  0001 C CNN
+F 2 "Connector_PinSocket_1.27mm:PinSocket_2x05_P1.27mm_Vertical" H 9700 3400 50  0001 C CNN
 F 3 "~" H 9700 3400 50  0001 C CNN
 	1    9700 3400
@@
 NoConn ~ 9500 3500
 $Comp
-L Connector_Generic:Conn_01x01 J12
-U 1 1 5C9F6723
-P 1450 2900
-F 0 "J12" H 1530 2942 50  0000 L CNN
-F 1 "Conn_01x01" H 1530 2851 50  0000 L CNN
-F 2 "E73:mouse-bite-2mm-slot" H 1450 2900 50  0001 C CNN
-F 3 "~" H 1450 2900 50  0001 C CNN
-	1    1450 2900
-	1    0    0    -1
-$EndComp
-NoConn ~ 1250 2900
-$Comp
-L Connector_Generic:Conn_01x01 J17
-U 1 1 5C9F6C0D
-P 2400 2650
-F 0 "J17" H 2480 2692 50  0000 L CNN
-F 1 "Conn_01x01" H 2480 2601 50  0000 L CNN
-F 2 "E73:mouse-bite-2mm-slot" H 2400 2650 50  0001 C CNN
-F 3 "~" H 2400 2650 50  0001 C CNN
-	1    2400 2650
-	1    0    0    -1
-$EndComp
-NoConn ~ 2200 2650
-$Comp
-L Connector_Generic:Conn_01x01 J18
-U 1 1 5C9F6C14
-P 2400 2900
-F 0 "J18" H 2480 2942 50  0000 L CNN
-F 1 "Conn_01x01" H 2480 2851 50  0000 L CNN
-F 2 "E73:mouse-bite-2mm-slot" H 2400 2900 50  0001 C CNN
-F 3 "~" H 2400 2900 50  0001 C CNN
-	1    2400 2900
-	1    0    0    -1
-$EndComp
-NoConn ~ 2200 2900
-$Comp
-L Connector_Generic:Conn_01x01 J13
-U 1 1 5C9F70F0
-P 1450 3300
-F 0 "J13" H 1530 3342 50  0000 L CNN
-F 1 "Conn_01x01" H 1530 3251 50  0000 L CNN
-F 2 "E73:mouse-bite-2mm-slot" H 1450 3300 50  0001 C CNN
-F 3 "~" H 1450 3300 50  0001 C CNN
-	1    1450 3300
-	1    0    0    -1
-$EndComp
-NoConn ~ 1250 3300
-$Comp
-L Connector_Generic:Conn_01x01 J14
-U 1 1 5C9F70F7
-P 1450 3550
-F 0 "J14" H 1530 3592 50  0000 L CNN
-F 1 "Conn_01x01" H 1530 3501 50  0000 L CNN
-F 2 "E73:mouse-bite-2mm-slot" H 1450 3550 50  0001 C CNN
-F 3 "~" H 1450 3550 50  0001 C CNN
-	1    1450 3550
-	1    0    0    -1
-$EndComp
-NoConn ~ 1250 3550
-$Comp
-L Connector_Generic:Conn_01x01 J19
-U 1 1 5C9F70FE
-P 2400 3300
-F 0 "J19" H 2480 3342 50  0000 L CNN
-F 1 "Conn_01x01" H 2480 3251 50  0000 L CNN
-F 2 "E73:mouse-bite-2mm-slot" H 2400 3300 50  0001 C CNN
-F 3 "~" H 2400 3300 50  0001 C CNN
-	1    2400 3300
-	1    0    0    -1
-$EndComp
-NoConn ~ 2200 3300
-$Comp
-L Connector_Generic:Conn_01x01 J20
-U 1 1 5C9F7105
-P 2400 3550
-F 0 "J20" H 2480 3592 50  0000 L CNN
-F 1 "Conn_01x01" H 2480 3501 50  0000 L CNN
-F 2 "E73:mouse-bite-2mm-slot" H 2400 3550 50  0001 C CNN
-F 3 "~" H 2400 3550 50  0001 C CNN
-	1    2400 3550
-	1    0    0    -1
-$EndComp
-NoConn ~ 2200 3550
-$Comp
-L Connector_Generic:Conn_01x01 J15
-U 1 1 5C9F766D
-P 1450 4000
-F 0 "J15" H 1530 4042 50  0000 L CNN
-F 1 "Conn_01x01" H 1530 3951 50  0000 L CNN
-F 2 "E73:mouse-bite-2mm-slot" H 1450 4000 50  0001 C CNN
-F 3 "~" H 1450 4000 50  0001 C CNN
-	1    1450 4000
-	1    0    0    -1
-$EndComp
-NoConn ~ 1250 4000
-$Comp
-L Connector_Generic:Conn_01x01 J16
-U 1 1 5C9F7674
-P 1450 4250
-F 0 "J16" H 1530 4292 50  0000 L CNN
-F 1 "Conn_01x01" H 1530 4201 50  0000 L CNN
-F 2 "E73:mouse-bite-2mm-slot" H 1450 4250 50  0001 C CNN
-F 3 "~" H 1450 4250 50  0001 C CNN
-	1    1450 4250
-	1    0    0    -1
-$EndComp
-NoConn ~ 1250 4250
-$Comp
-L Connector_Generic:Conn_01x01 J21
-U 1 1 5C9F767B
-P 2400 4000
-F 0 "J21" H 2480 4042 50  0000 L CNN
-F 1 "Conn_01x01" H 2480 3951 50  0000 L CNN
-F 2 "E73:mouse-bite-2mm-slot" H 2400 4000 50  0001 C CNN
-F 3 "~" H 2400 4000 50  0001 C CNN
-	1    2400 4000
-	1    0    0    -1
-$EndComp
-NoConn ~ 2200 4000
-$Comp
-L Connector_Generic:Conn_01x01 J22
-U 1 1 5C9F7682
-P 2400 4250
-F 0 "J22" H 2480 4292 50  0000 L CNN
-F 1 "Conn_01x01" H 2480 4201 50  0000 L CNN
-F 2 "E73:mouse-bite-2mm-slot" H 2400 4250 50  0001 C CNN
-F 3 "~" H 2400 4250 50  0001 C CNN
-	1    2400 4250
-	1    0    0    -1
-$EndComp
-NoConn ~ 2200 4250
+L Connector_Generic:Conn_02x05_Odd_Even J5
+U 1 1 5DF01131
+P 8800 1550
+F 0 "J5" H 8850 1967 50  0000 C CNN
+F 1 "Cortex Debug 10-pin connector" H 8850 1876 50  0000 C CNN
+F 2 "Connector_PinHeader_1.27mm:PinHeader_2x05_P1.27mm_Vertical" H 8800 1550 50  0001 C CNN
+F 3 "~" H 8800 1550 50  0001 C CNN
+	1    8800 1550
+	1    0    0    -1
+$EndComp
 $EndSCHEMATC
