File: BlueMicro2.1a/EByte_E73.sch (KiCad schematic (older format))
At the start: 28 parts, among them J1 USB_OTG, J2 Serial Connector, J3 Conn_01x02, Q1 DMG3415U, U1 E73-2G4M04S, U2 ProMicro, U3 AP2112K-3.3, U4 CH340C, U6 TP4056

Commit message: updated to 2.1a
Parts:
- removed JP1: JUMPER-SMT_2_NO, E73:SolderJumperSingle, symbol EByte_E73-rescue:JUMPER-SMT_2_NO
- added C10, C11, C12: 100nF, Resistor_SMD:R_0805_2012Metric, symbol Device:C_Small
- added D2, D3: D, Diode_SMD:D_SOD-123, symbol Device:D
- added D4: BLUE, LED_SMD:LED_0805_2012Metric, symbol Device:LED
- added D5, D6: RED, LED_SMD:LED_0805_2012Metric, symbol Device:LED
- added R10, R8, R9: 1k, Resistor_SMD:R_0805_2012Metric, symbol Device:R
- added R7: JUMP, Resistor_SMD:R_0402_1005Metric, symbol Device:R
- C1, C2, C3, C4, C5, C6, C7, C8, C9: footprint Capacitors_SMD:C_0805_HandSoldering -> Resistor_SMD:R_0805_2012Metric
- D1: footprint Diodes_SMD:D_SOD-123 -> Diode_SMD:D_SOD-123
- L1: footprint Inductors_SMD:L_0805_HandSoldering -> Inductor_SMD:L_0805_2012Metric
- R1, R2, R3, R4, R5, R6: footprint Resistors_SMD:R_0805_HandSoldering -> Resistor_SMD:R_0805_2012Metric
- U3: footprint TO_SOT_Packages_SMD:SOT-23-5_HandSoldering -> Package_TO_SOT_SMD:SOT-23-5
Connections:
- net labels added: LED1, LED2
- net labels removed: P0.17, P0.19
- wire segments 180 -> 204
- no-connect marks 10 -> 9
