File: 4x4_backpack/4x4_backpack_nrf52840/4x4_backpack.kicad_pcb (KiCad board)
At the start: 2 copper layers, 76.2 x 76.2 mm, 49 parts, among them J1 Conn_01x04, J10 TC2050, J11 Conn_01x01, J12 Conn_01x01, J13 Conn_01x01, J14 Conn_01x01, J15 Conn_01x01, J16 Conn_01x01, J17 USB_B_Micro, J2 Conn_01x04, J3 Conn_01x04, J4 Conn_01x04, J5 Conn_01x04, J6 Conn_01x04, J7 Conn_01x04, J8 Conn_01x04, J9 Conn_01x04, Q1 P5102FM, SW1 SW_SPDT, SW2 RESET, U1 E73-2G4M08S1C, U2 TP4056, U3 AP2112K-3.3, Y1 32.768kHz

Commit message: adding bunch of stuff (sorry for the massive changes)
Parts:
- added J18: Conn_01x02, Connector_PinHeader_2.54mm:PinHeader_1x02_P2.54mm_Vertical, F.Cu at (118.7, 130.9)
Routing:
- net Net-(E1-Pad1): track 47.5 -> 50.1 mm
- net GND: track 166.6 -> 168.7 mm
- net Net-(C2-Pad1): track 93.1 -> 91.8 mm
Other:
- board text added: "2020-05-09"
- board text added: "Replace R3 with 10k for Lipo"
- board text added: "VBatt"
- board text added: "gnd"
Changed lines of the file:
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@@
   (general
     (thickness 1.6)
-    (drawings 38)
-    (tracks 684)
+    (drawings 42)
+    (tracks 687)
     (zones 0)
-    (modules 49)
+    (modules 50)
     (nets 47)
   )
@@
   )
   (setup
-    (last_trace_width 0.25)
+    (last_trace_width 1)
     (user_trace_width 0.5)
     (user_trace_width 1)
@@
     )
   )
+  (module Connector_PinHeader_2.54mm:PinHeader_1x02_P2.54mm_Vertical (layer F.Cu)
+    (at 118.745 130.937)
+    (descr "Through hole straight pin header, 1x02, 2.54mm pitch, single row")
+    (tags "Through hole pin header THT 1x02 2.54mm single row")
+    (fp_text reference J18 (at 0 -2.33) (layer F.SilkS) hide
+      (effects (font (size 1 1) (thickness 0.15)))
+    )
+    (fp_text value Conn_01x02 (at 0 4.87) (layer F.Fab)
+      (effects (font (size 1 1) (thickness 0.15)))
+    )
+    (fp_line (start -0.635 -1.27) (end 1.27 -1.27) (layer F.Fab) (width 0.1))
+    (fp_line (start 1.27 -1.27) (end 1.27 3.81) (layer F.Fab) (width 0.1))
+    (fp_line (start 1.27 3.81) (end -1.27 3.81) (layer F.Fab) (width 0.1))
+    (fp_line (start -1.27 3.81) (end -1.27 -0.635) (layer F.Fab) (width 0.1))
+    (fp_line (start -1.27 -0.635) (end -0.635 -1.27) (layer F.Fab) (width 0.1))
+    (fp_line (start -1.33 3.87) (end 1.33 3.87) (layer F.SilkS) (width 0.12))
+    (fp_line (start -1.33 1.27) (end -1.33 3.87) (layer F.SilkS) (width 0.12))
+    (fp_line (start 1.33 1.27) (end 1.33 3.87) (layer F.SilkS) (width 0.12))
+    (fp_line (start -1.33 1.27) (end 1.33 1.27) (layer F.SilkS) (width 0.12))
+    (fp_line (start -1.33 0) (end -1.33 -1.33) (layer F.SilkS) (width 0.12))
+    (fp_line (start -1.33 -1.33) (end 0 -1.33) (layer F.SilkS) (width 0.12))
+    (fp_line (start -1.8 -1.8) (end -1.8 4.35) (layer F.CrtYd) (width 0.05))
+    (fp_line (start -1.8 4.35) (end 1.8 4.35) (layer F.CrtYd) (width 0.05))
+    (fp_line (start 1.8 4.35) (end 1.8 -1.8) (layer F.CrtYd) (width 0.05))
+    (fp_line (start 1.8 -1.8) (end -1.8 -1.8) (layer F.CrtYd) (width 0.05))
+    (fp_text user %R (at 0 1.27 90) (layer F.Fab)
+      (effects (font (size 1 1) (thickness 0.15)))
+    )
+    (pad 1 thru_hole rect (at 0 0) (size 1.7 1.7) (drill 1) (layers *.Cu *.Mask)
+      (net 21 GND))
+    (pad 2 thru_hole oval (at 0 2.54) (size 1.7 1.7) (drill 1) (layers *.Cu *.Mask)
+      (net 25 "Net-(E1-Pad1)"))
+    (model ${KISYS3DMOD}/Connector_PinHeader_2.54mm.3dshapes/PinHeader_1x02_P2.54mm_Vertical.wrl
+      (at (xyz 0 0 0))
+      (scale (xyz 1 1 1))
+      (rotate (xyz 0 0 0))
+    )
+  )
+  (gr_text gnd (at 117.983 128.905) (layer F.SilkS)
+    (effects (font (size 1 1) (thickness 0.1)))
+  )
+  (gr_text "Replace R3 with \n10k for Lipo" (at 124.968 99.187) (layer F.SilkS)
+    (effects (font (size 1 1) (thickness 0.1)))
+  )
+  (gr_text VBatt (at 118.745 135.636) (layer F.SilkS)
+    (effects (font (size 1 1) (thickness 0.1)))
+  )
+  (gr_text 2020-05-09 (at 128.27 88.9) (layer F.SilkS)
+    (effects (font (size 1.5 1.5) (thickness 0.3)))
+  )
   (gr_text "Use \nBlueMicro_BLE \nFirmware" (at 125.984 109.347) (layer F.SilkS)
     (effects (font (size 1.5 1.5) (thickness 0.3)))
@@
     (effects (font (size 1.5 1.5) (thickness 0.3)))
   )
-  (gr_text "USE LIR2032 ONLY" (at 130.8862 150.3426) (layer F.SilkS)
+  (gr_text "USE LIR2032 ONLY" (at 131.318 143.637) (layer F.SilkS)
     (effects (font (size 1.5 1.5) (thickness 0.3)))
   )
@@
   (segment (start 90.76 146.63) (end 95.81 146.63) (width 0.25) (layer F.Cu) (net 21) (status 20))
   (segment (start 89.61 146.63) (end 90.76 146.63) (width 0.25) (layer F.Cu) (net 21) (status 10))
-  (segment (start 147.701 133.477) (end 109.601 133.477) (width 0.25) (layer B.Cu) (net 21) (status 30))
   (segment (start 102.34401 102.235) (end 102.34401 100.09399) (width 0.25) (layer F.Cu) (net 21) (status 10))
   (segment (start 102.799 99.639) (end 102.799 97.955) (width 0.25) (layer F.Cu) (net 21) (status 20))
@@
   (via (at 111.5 90.25) (size 0.8) (drill 0.4) (layers F.Cu B.Cu) (net 21))
   (via (at 86.75 86) (size 0.8) (drill 0.4) (layers F.Cu B.Cu) (net 21))
-  (segment (start 113.665 113.448) (end 113.665 114.898) (width 1) (layer B.Cu) (net 22) (status 20))
+  (segment (start 112.141 136.017) (end 109.601 133.477) (width 0.25) (layer B.Cu) (net 21))
+  (segment (start 147.701 133.477) (end 145.161 136.017) (width 0.25) (layer B.Cu) (net 21))
+  (segment (start 145.161 136.017) (end 112.141 136.017) (width 0.25) (layer B.Cu) (net 21))
   (segment (start 109.51 143.62) (end 113.665 139.465) (width 1) (layer F.Cu) (net 22))
   (segment (start 109.51 145.245) (end 109.51 143.62) (width 1) (layer F.Cu) (net 22) (status 10))
-  (segment (start 113.665 114.808) (end 113.665 113.448) (width 0.25) (layer F.Cu) (net 22))
   (segment (start 94.811001 114.808) (end 113.665 114.808) (width 0.25) (layer F.Cu) (net 22))
   (segment (start 87.884 107.205999) (end 87.884 107.880999) (width 0.25) (layer F.Cu) (net 22) (status 10))
@@
   (segment (start 117.33 118.491) (end 116.655 118.491) (width 1) (layer F.Cu) (net 22) (status 10))
   (segment (start 113.665 139.465) (end 113.665 118.491) (width 1) (layer F.Cu) (net 22))
-  (segment (start 113.665 118.491) (end 113.665 113.448) (width 1) (layer F.Cu) (net 22))
   (segment (start 117.33 118.491) (end 117.33 116.858) (width 1) (layer F.Cu) (net 22) (status 10))
   (segment (start 133.005 105.41) (end 134.78 105.41) (width 1) (layer F.Cu) (net 22) (status 20))
@@
   (segment (start 120.505 116.858) (end 131.953 105.41) (width 1) (layer F.Cu) (net 22))
   (segment (start 117.33 116.858) (end 120.505 116.858) (width 1) (layer F.Cu) (net 22))
+  (segment (start 113.665 111.998) (end 113.665 114.808) (width 1) (layer F.Cu) (net 22))
+  (segment (start 113.665 114.808) (end 113.665 118.491) (width 1) (layer F.Cu) (net 22))
   (segment (start 104.39401 99.29201) (end 104.39401 102.235) (width 0.25) (layer F.Cu) (net 23) (status 20))
   (segment (start 104.069 97.955) (end 104.069 98.967) (width 0.25) (layer F.Cu) (net 23) (status 10))
@@
   (segment (start 95.81 141.44) (end 99.75 137.5) (width 0.25) (layer F.Cu) (net 24))
   (segment (start 95.81 142.93) (end 95.81 141.44) (width 0.25) (layer F.Cu) (net 24))
-  (segment (start 118.618 142.337) (end 118.618 140.462) (width 0.25) (layer F.Cu) (net 25) (status 20))
   (segment (start 115.668 140.462) (end 118.618 140.462) (width 1) (layer F.Cu) (net 25) (status 20))
   (segment (start 112.51 145.245) (end 112.51 143.62) (width 1) (layer F.Cu) (net 25) (status 10))
@@
   (segment (start 118.618 140.462) (end 118.618 137.837) (width 1) (layer F.Cu) (net 25) (status 10))
   (segment (start 118.618 137.837) (end 126.661 129.794) (width 1) (layer F.Cu) (net 25))
+  (segment (start 118.618 140.462) (end 118.618 140.462) (width 0.25) (layer F.Cu) (net 25) (status 20))
+  (segment (start 118.745 137.71) (end 118.745 133.477) (width 1) (layer F.Cu) (net 25))
+  (segment (start 118.618 137.837) (end 118.745 137.71) (width 1) (layer F.Cu) (net 25))
   (segment (start 123.19 85.09) (end 123.19 85.725) (width 0.25) (layer B.Cu) (net 26) (status 30))
   (segment (start 134.239 94.185225) (end 134.239 94.742) (width 0.25) (layer B.Cu) (net 26) (status 20))
