File: 4x4_backpack/4x4_backpack_nrf52840/4x4_backpack.sch (KiCad schematic (older format))
At the start: 49 parts, among them J1 Conn_01x04, J10 TC2050, J11 Conn_01x01, J12 Conn_01x01, J13 Conn_01x01, J14 Conn_01x01, J15 Conn_01x01, J16 Conn_01x01, J17 USB_B_Micro, J2 Conn_01x04, J3 Conn_01x04, J4 Conn_01x04, J5 Conn_01x04, J6 Conn_01x04, J7 Conn_01x04, J8 Conn_01x04, J9 Conn_01x04, Q1 P5102FM, SW1 SW_SPDT, SW2 RESET, U1 E73-2G4M08S1C, U2 TP4056, U3 AP2112K-3.3, Y1 32.768kHz

Commit message: adding bunch of stuff (sorry for the massive changes)
Parts:
- added J18: Conn_01x02, Connector_PinHeader_2.54mm:PinHeader_1x02_P2.54mm_Vertical, symbol Connector_Generic:Conn_01x02
Connections:
- wire segments 219 -> 226
Changed lines of the file:
@@
 EELAYER 26 0
 EELAYER END
-$Descr A4 11693 8268
+$Descr USLetter 11000 8500
 encoding utf-8
 Sheet 1 1
-Title ""
-Date ""
+Title "4x4Backpack NRF52840"
+Date "2020-03-14"
 Rev ""
 Comp ""
@@
 L E73:SW_PUSH SW2
 U 1 1 5BBF7215
-P 9850 5850
-F 0 "SW2" H 9850 6105 50  0000 C CNN
-F 1 "RESET" H 9850 6014 50  0000 C CNN
-F 2 "E73:SW_TACT_ALPS_SKQGABE010" H 9850 5850 60  0001 C CNN
-F 3 "" H 9850 5850 60  0000 C CNN
-	1    9850 5850
+P 9150 6100
+F 0 "SW2" H 9150 6355 50  0000 C CNN
+F 1 "RESET" H 9150 6264 50  0000 C CNN
+F 2 "E73:SW_TACT_ALPS_SKQGABE010" H 9150 6100 60  0001 C CNN
+F 3 "" H 9150 6100 60  0000 C CNN
+	1    9150 6100
 	1    0    0    -1
 $EndComp
@@
 L power:VCC #PWR07
 U 1 1 5BBF89FC
-P 10450 5400
-F 0 "#PWR07" H 10450 5250 50  0001 C CNN
-F 1 "VCC" H 10467 5573 50  0000 C CNN
-F 2 "" H 10450 5400 50  0001 C CNN
-F 3 "" H 10450 5400 50  0001 C CNN
-	1    10450 5400
+P 9750 5650
+F 0 "#PWR07" H 9750 5500 50  0001 C CNN
+F 1 "VCC" H 9767 5823 50  0000 C CNN
+F 2 "" H 9750 5650 50  0001 C CNN
+F 3 "" H 9750 5650 50  0001 C CNN
+	1    9750 5650
 	1    0    0    -1
 $EndComp
@@
 L power:GND #PWR06
 U 1 1 5BBF8A67
-P 9150 6200
-F 0 "#PWR06" H 9150 5950 50  0001 C CNN
-F 1 "GND" H 9155 6027 50  0000 C CNN
-F 2 "" H 9150 6200 50  0001 C CNN
-F 3 "" H 9150 6200 50  0001 C CNN
-	1    9150 6200
+P 8450 6450
+F 0 "#PWR06" H 8450 6200 50  0001 C CNN
+F 1 "GND" H 8455 6277 50  0000 C CNN
+F 2 "" H 8450 6450 50  0001 C CNN
+F 3 "" H 8450 6450 50  0001 C CNN
+	1    8450 6450
 	1    0    0    -1
 $EndComp
@@
 L Device:R R1
 U 1 1 5BBF8AB1
-P 10450 5650
-F 0 "R1" H 10520 5696 50  0000 L CNN
-F 1 "10k" H 10520 5605 50  0000 L CNN
-F 2 "Resistor_SMD:R_0805_2012Metric_Pad1.15x1.40mm_HandSolder" V 10380 5650 50  0001 C CNN
-F 3 "~" H 10450 5650 50  0001 C CNN
-	1    10450 5650
+P 9750 5900
+F 0 "R1" H 9820 5946 50  0000 L CNN
+F 1 "10k" H 9820 5855 50  0000 L CNN
+F 2 "Resistor_SMD:R_0805_2012Metric_Pad1.15x1.40mm_HandSolder" V 9680 5900 50  0001 C CNN
+F 3 "~" H 9750 5900 50  0001 C CNN
+	1    9750 5900
 	1    0    0    -1
 $EndComp
@@
 	7050 3300 7050 3350
 Wire Wire Line
-	9550 5850 9150 5850
-Wire Wire Line
-	9150 5850 9150 6200
-Wire Wire Line
-	10450 5400 10450 5500
-Wire Wire Line
-	10450 5800 10450 5850
-Wire Wire Line
-	10450 5850 10150 5850
-Wire Wire Line
-	10450 5850 10650 5850
-Connection ~ 10450 5850
-Text GLabel 10650 5850 2    50   Input ~ 0
+	8850 6100 8450 6100
+Wire Wire Line
+	8450 6100 8450 6450
+Wire Wire Line
+	9750 5650 9750 5750
+Wire Wire Line
+	9750 6050 9750 6100
+Wire Wire Line
+	9750 6100 9450 6100
+Wire Wire Line
+	9750 6100 9950 6100
+Connection ~ 9750 6100
+Text GLabel 9950 6100 2    50   Input ~ 0
 RESET
 $Comp
@@
 	2150 7000 1750 7000
 Wire Wire Line
-	850  7100 850  7000
+	850  7100 850  7050
 Wire Wire Line
 	1850 6500 2150 6500
@@
 Text GLabel 9150 3100 2    50   Input ~ 0
 WS2812
+Wire Wire Line
+	450  6600 850  6600
+Connection ~ 850  6600
+Wire Wire Line
+	450  7150 600  7150
+Wire Wire Line
+	600  7150 600  7050
+Wire Wire Line
+	600  7050 850  7050
+Connection ~ 850  7050
+Wire Wire Line
+	850  7050 850  7000
+$Comp
+L Connector_Generic:Conn_01x02 J18
+U 1 1 5ECB4A54
+P 250 6900
+F 0 "J18" H 170 6575 50  0000 C CNN
+F 1 "Conn_01x02" H 170 6666 50  0000 C CNN
+F 2 "Connector_PinHeader_2.54mm:PinHeader_1x02_P2.54mm_Vertical" H 250 6900 50  0001 C CNN
+F 3 "~" H 250 6900 50  0001 C CNN
+	1    250  6900
+	-1   0    0    1
+$EndComp
+Wire Wire Line
+	450  6600 450  6800
+Wire Wire Line
+	450  6900 450  7150
 $EndSCHEMATC
