File: BlueMicro840/BlueMicro840.sch (KiCad schematic (older format))
At the start: 36 parts, among them J2 Conn_01x02_Male, J3 DNP, Q1 SI2301CDS-T1-GE3, U1 AP2112K-3.3TRG1, U2 ProMicro, U3 AP2112K-3.3TRG1, U4 TP4054ST, U5 E73-2G4M08S1C-52840, Y2 32,768

Commit message: adding BOM to Docs
Parts:
- J3: LCSC (none) -> C165948
- L1: LCSC (none) -> C1046
Connections:
- net labels added: 1.02
- net labels removed: DFU
Changed lines of the file:
@@
 F 2 "Inductor_SMD:L_0805_2012Metric" H 3450 3150 50  0001 C CNN
 F 3 "~" H 3450 3150 50  0001 C CNN
+F 4 "C1046" H 3450 3150 50  0001 C CNN "LCSC"
 	1    3450 3150
 	1    0    0    -1
@@
 	4500 7350 4500 7400
 Text GLabel 3300 1650 2    60   Input ~ 0
-DFU
+1.02
 Wire Wire Line
 	3000 1650 3300 1650
@@
 $EndComp
 Text GLabel 1350 4100 0    60   Input ~ 0
-DFU
+1.02
 Wire Wire Line
 	2000 6300 2000 6250
@@
 F 2 "footprints:HRO-TYPE-C-31-M-12-C165948" H 7700 5550 50  0001 C CNN
 F 3 "" H 7700 5550 50  0001 C CNN
+F 4 "C165948" H 7550 5550 50  0001 C CNN "LCSC"
 	1    7550 5550
 	1    0    0    -1
