File: BlueMacro840/BlueMacro.sch (KiCad schematic (older format))
At the start: 33 parts, among them J1 Conn_01x02, J3 USB_C_Receptacle, Q1 SI2301CDS-T1-GE3, U1 TP4054ST, U2 E73-2G4M08S1C, U3 AP2112K-3.3, U4 Micro, U5 AP2112K-3.3, Y1 32.768kHz

Commit message: updates to BlueMacro840
Parts:
- C1, C2: footprint Capacitor_SMD:C_0402_1005Metric -> Capacitor_SMD:C_0603_1608Metric; LCSC C1555 -> C1653
- C3, C4, C5: footprint Capacitor_SMD:C_0402_1005Metric -> Capacitor_SMD:C_0603_1608Metric; LCSC C15525 -> C19702
- C6: footprint Capacitor_SMD:C_0402_1005Metric -> Capacitor_SMD:C_0603_1608Metric; LCSC C1523 -> C1588
- D2: value 16-213/GHC-YR1S1/3T -> 19-217/GHC-YR1S2/3T; footprint LED_SMD:LED_0402_1005Metric -> LED_SMD:LED_0603_1608Metric; LCSC C74338 -> C72043
- D3: value 16-213SURC/S530-A4/TR8 -> KT-0603R; footprint LED_SMD:LED_0402_1005Metric -> LED_SMD:LED_0603_1608Metric; LCSC C74339 -> C2286
- D4: value FC-F1005BK-470G5 -> 19-217/BHC-ZL1M2RY/3T; footprint LED_SMD:LED_0402_1005Metric -> LED_SMD:LED_0603_1608Metric; LCSC C130724 -> C72041
- R1: footprint Resistor_SMD:R_0402_1005Metric -> Resistor_SMD:R_0603_1608Metric; LCSC C25741 -> C25803
- R2: footprint Resistor_SMD:R_0402_1005Metric -> Resistor_SMD:R_0603_1608Metric; LCSC C25744 -> C25804
- R3, R7, R8: footprint Resistor_SMD:R_0402_1005Metric -> Resistor_SMD:R_0603_1608Metric; LCSC C11702 -> C21190
- R4: footprint Resistor_SMD:R_0402_1005Metric -> Resistor_SMD:R_0603_1608Metric; LCSC C29263 -> C23250
- R5: footprint Resistor_SMD:R_0402_1005Metric -> Resistor_SMD:R_0603_1608Metric; LCSC C11512 -> C22976
- R6, R9: footprint Resistor_SMD:R_0402_1005Metric -> Resistor_SMD:R_0603_1608Metric; LCSC C25905 -> C23186
- U3, U5: value AP2112K-3.3 -> AP2112K-3.3TRG1
Changed lines of the file:
@@
 P 3150 6650
 F 0 "U3" H 3125 6687 60  0000 C CNN
-F 1 "AP2112K-3.3" H 3125 6581 60  0000 C CNN
+F 1 "AP2112K-3.3TRG1" H 3125 6581 60  0000 C CNN
 F 2 "Package_TO_SOT_SMD:SOT-23-5" H 3150 5950 60  0001 C CNN
 F 3 "" H 3150 5950 60  0001 C CNN
@@
 F 0 "R4" H 4720 5596 50  0000 L CNN
 F 1 "806k" H 4720 5505 50  0000 L CNN
-F 2 "Resistor_SMD:R_0402_1005Metric" V 4580 5550 50  0001 C CNN
+F 2 "Resistor_SMD:R_0603_1608Metric" V 4580 5550 50  0001 C CNN
 F 3 "~" H 4650 5550 50  0001 C CNN
-F 4 "C29263" H 4650 5550 50  0001 C CNN "LCSC"
+F 4 "C23250" H 4650 5550 50  0001 C CNN "LCSC"
 	1    4650 5550
 	1    0    0    -1
@@
 F 0 "R5" H 4720 6046 50  0000 L CNN
 F 1 "2M" H 4720 5955 50  0000 L CNN
-F 2 "Resistor_SMD:R_0402_1005Metric" V 4580 6000 50  0001 C CNN
+F 2 "Resistor_SMD:R_0603_1608Metric" V 4580 6000 50  0001 C CNN
 F 3 "~" H 4650 6000 50  0001 C CNN
-F 4 "C11512" H 4650 6000 50  0001 C CNN "LCSC"
+F 4 "C22976" H 4650 6000 50  0001 C CNN "LCSC"
 	1    4650 6000
 	1    0    0    -1
@@
 F 0 "C6" H 4242 6046 50  0000 L CNN
 F 1 "1nF" H 4242 5955 50  0000 L CNN
-F 2 "Capacitor_SMD:C_0402_1005Metric" H 4150 6000 50  0001 C CNN
+F 2 "Capacitor_SMD:C_0603_1608Metric" H 4150 6000 50  0001 C CNN
 F 3 "~" H 4150 6000 50  0001 C CNN
-F 4 "C1523" H 4150 6000 50  0001 C CNN "LCSC"
+F 4 "C1588" H 4150 6000 50  0001 C CNN "LCSC"
 	1    4150 6000
 	1    0    0    -1
@@
 F 0 "C3" H 1892 7196 50  0000 L CNN
 F 1 "10uF" H 1892 7105 50  0000 L CNN
-F 2 "Capacitor_SMD:C_0402_1005Metric" H 1800 7150 50  0001 C CNN
+F 2 "Capacitor_SMD:C_0603_1608Metric" H 1800 7150 50  0001 C CNN
 F 3 "~" H 1800 7150 50  0001 C CNN
-F 4 "C15525" H 1800 7150 50  0001 C CNN "LCSC"
+F 4 "C19702" H 1800 7150 50  0001 C CNN "LCSC"
 	1    1800 7150
 	1    0    0    -1
@@
 F 0 "R1" H 1120 7196 50  0000 L CNN
 F 1 "100k" H 1120 7105 50  0000 L CNN
-F 2 "Resistor_SMD:R_0402_1005Metric" V 980 7150 50  0001 C CNN
+F 2 "Resistor_SMD:R_0603_1608Metric" V 980 7150 50  0001 C CNN
 F 3 "~" H 1050 7150 50  0001 C CNN
-F 4 "C25741" H 1050 7150 50  0001 C CNN "LCSC"
+F 4 "C25803" H 1050 7150 50  0001 C CNN "LCSC"
 	1    1050 7150
 	1    0    0    -1
@@
 F 0 "C5" H 4142 7096 50  0000 L CNN
 F 1 "10uF" H 4142 7005 50  0000 L CNN
-F 2 "Capacitor_SMD:C_0402_1005Metric" H 4050 7050 50  0001 C CNN
+F 2 "Capacitor_SMD:C_0603_1608Metric" H 4050 7050 50  0001 C CNN
 F 3 "~" H 4050 7050 50  0001 C CNN
-F 4 "C15525" H 4050 7050 50  0001 C CNN "LCSC"
+F 4 "C19702" H 4050 7050 50  0001 C CNN "LCSC"
 	1    4050 7050
 	1    0    0    -1
@@
 F 0 "R2" V 1993 5750 50  0000 C CNN
 F 1 "10k" V 2084 5750 50  0000 C CNN
-F 2 "Resistor_SMD:R_0402_1005Metric" V 2130 5750 50  0001 C CNN
+F 2 "Resistor_SMD:R_0603_1608Metric" V 2130 5750 50  0001 C CNN
 F 3 "~" H 2200 5750 50  0001 C CNN
-F 4 "C25744" V 2200 5750 50  0001 C CNN "LCSC"
+F 4 "C25804" V 2200 5750 50  0001 C CNN "LCSC"
 	1    2200 5750
 	0    1    1    0
@@
 F 0 "R3" V 1993 6100 50  0000 C CNN
 F 1 "1k" V 2084 6100 50  0000 C CNN
-F 2 "Resistor_SMD:R_0402_1005Metric" V 2130 6100 50  0001 C CNN
+F 2 "Resistor_SMD:R_0603_1608Metric" V 2130 6100 50  0001 C CNN
 F 3 "~" H 2200 6100 50  0001 C CNN
-F 4 "C11702" V 2200 6100 50  0001 C CNN "LCSC"
+F 4 "C21190" V 2200 6100 50  0001 C CNN "LCSC"
 	1    2200 6100
 	0    1    1    0
@@
 P 1700 6100
 F 0 "D2" H 1692 5845 50  0000 C CNN
-F 1 "16-213/GHC-YR1S1/3T" H 1692 5936 50  0000 C CNN
-F 2 "LED_SMD:LED_0402_1005Metric" H 1700 6100 50  0001 C CNN
+F 1 "19-217/GHC-YR1S2/3T" H 1692 5936 50  0000 C CNN
+F 2 "LED_SMD:LED_0603_1608Metric" H 1700 6100 50  0001 C CNN
 F 3 "~" H 1700 6100 50  0001 C CNN
-F 4 "C74338" H 1700 6100 50  0001 C CNN "LCSC"
+F 4 "C72043" H 1700 6100 50  0001 C CNN "LCSC"
 	1    1700 6100
 	-1   0    0    1
@@
 F 0 "C4" H 3442 5496 50  0000 L CNN
 F 1 "10uF" H 3442 5405 50  0000 L CNN
-F 2 "Capacitor_SMD:C_0402_1005Metric" H 3350 5450 50  0001 C CNN
+F 2 "Capacitor_SMD:C_0603_1608Metric" H 3350 5450 50  0001 C CNN
 F 3 "~" H 3350 5450 50  0001 C CNN
-F 4 "C15525" H 3350 5450 50  0001 C CNN "LCSC"
+F 4 "C19702" H 3350 5450 50  0001 C CNN "LCSC"
 	1    3350 5450
 	1    0    0    -1
@@
 F 0 "R6" H 9680 1604 50  0000 R CNN
 F 1 "5.1k" H 9680 1695 50  0000 R CNN
-F 2 "Resistor_SMD:R_0402_1005Metric" V 9680 1650 50  0001 C CNN
+F 2 "Resistor_SMD:R_0603_1608Metric" V 9680 1650 50  0001 C CNN
 F 3 "~" H 9750 1650 50  0001 C CNN
-F 4 "C25905" H 9750 1650 50  0001 C CNN "LCSC"
+F 4 "C23186" H 9750 1650 50  0001 C CNN "LCSC"
 	1    9750 1650
 	-1   0    0    1
@@
 F 0 "R9" H 10030 1604 50  0000 R CNN
 F 1 "5.1k" H 10030 1695 50  0000 R CNN
-F 2 "Resistor_SMD:R_0402_1005Metric" V 10030 1650 50  0001 C CNN
+F 2 "Resistor_SMD:R_0603_1608Metric" V 10030 1650 50  0001 C CNN
 F 3 "~" H 10100 1650 50  0001 C CNN
-F 4 "C25905" H 10100 1650 50  0001 C CNN "LCSC"
+F 4 "C23186" H 10100 1650 50  0001 C CNN "LCSC"
 	1    10100 1650
 	-1   0    0    1
@@
 P 9300 5150
 F 0 "D3" H 9292 4895 50  0000 C CNN
-F 1 "16-213SURC/S530-A4/TR8" H 9292 4986 50  0000 C CNN
-F 2 "LED_SMD:LED_0402_1005Metric" H 9300 5150 50  0001 C CNN
+F 1 "KT-0603R" H 9292 4986 50  0000 C CNN
+F 2 "LED_SMD:LED_0603_1608Metric" H 9300 5150 50  0001 C CNN
 F 3 "~" H 9300 5150 50  0001 C CNN
-F 4 "C74339" H 9300 5150 50  0001 C CNN "LCSC"
+F 4 "C2286" H 9300 5150 50  0001 C CNN "LCSC"
 	1    9300 5150
 	-1   0    0    1
@@
 F 0 "R7" V 9543 5150 50  0000 C CNN
 F 1 "1k" V 9634 5150 50  0000 C CNN
-F 2 "Resistor_SMD:R_0402_1005Metric" V 9680 5150 50  0001 C CNN
+F 2 "Resistor_SMD:R_0603_1608Metric" V 9680 5150 50  0001 C CNN
 F 3 "~" H 9750 5150 50  0001 C CNN
-F 4 "C11702" V 9750 5150 50  0001 C CNN "LCSC"
+F 4 "C21190" V 9750 5150 50  0001 C CNN "LCSC"
 	1    9750 5150
 	0    1    1    0
@@
 F 0 "R8" V 9543 5500 50  0000 C CNN
 F 1 "1k" V 9634 5500 50  0000 C CNN
-F 2 "Resistor_SMD:R_0402_1005Metric" V 9680 5500 50  0001 C CNN
+F 2 "Resistor_SMD:R_0603_1608Metric" V 9680 5500 50  0001 C CNN
 F 3 "~" H 9750 5500 50  0001 C CNN
-F 4 "C11702" V 9750 5500 50  0001 C CNN "LCSC"
+F 4 "C21190" V 9750 5500 50  0001 C CNN "LCSC"
 	1    9750 5500
 	0    1    1    0
@@
 P 9300 5500
 F 0 "D4" H 9292 5245 50  0000 C CNN
-F 1 "FC-F1005BK-470G5" H 9292 5336 50  0000 C CNN
-F 2 "LED_SMD:LED_0402_1005Metric" H 9300 5500 50  0001 C CNN
+F 1 "19-217/BHC-ZL1M2RY/3T" H 9292 5336 50  0000 C CNN
+F 2 "LED_SMD:LED_0603_1608Metric" H 9300 5500 50  0001 C CNN
 F 3 "~" H 9300 5500 50  0001 C CNN
-F 4 "C130724" H 9300 5500 50  0001 C CNN "LCSC"
+F 4 "C72041" H 9300 5500 50  0001 C CNN "LCSC"
 	1    9300 5500
 	-1   0    0    1
@@
 F 0 "C1" V 921 1950 50  0000 C CNN
 F 1 "22pF" V 1012 1950 50  0000 C CNN
-F 2 "Capacitor_SMD:C_0402_1005Metric" H 1150 1950 50  0001 C CNN
+F 2 "Capacitor_SMD:C_0603_1608Metric" H 1150 1950 50  0001 C CNN
 F 3 "~" H 1150 1950 50  0001 C CNN
-F 4 "C1555" V 1150 1950 50  0001 C CNN "LCSC"
+F 4 "C1653" V 1150 1950 50  0001 C CNN "LCSC"
 	1    1150 1950
 	0    1    1    0
@@
 F 0 "C2" V 921 2350 50  0000 C CNN
 F 1 "22pF" V 1012 2350 50  0000 C CNN
-F 2 "Capacitor_SMD:C_0402_1005Metric" H 1150 2350 50  0001 C CNN
+F 2 "Capacitor_SMD:C_0603_1608Metric" H 1150 2350 50  0001 C CNN
 F 3 "~" H 1150 2350 50  0001 C CNN
-F 4 "C1555" V 1150 2350 50  0001 C CNN "LCSC"
+F 4 "C1653" V 1150 2350 50  0001 C CNN "LCSC"
 	1    1150 2350
 	0    1    1    0
@@
 P 5650 6650
 F 0 "U5" H 5625 6687 60  0000 C CNN
-F 1 "AP2112K-3.3" H 5625 6581 60  0000 C CNN
+F 1 "AP2112K-3.3TRG1" H 5625 6581 60  0000 C CNN
 F 2 "Package_TO_SOT_SMD:SOT-23-5" H 5650 5950 60  0001 C CNN
 F 3 "" H 5650 5950 60  0001 C CNN

Commit message: adding BOM to Docs
Parts:
- J3: LCSC (none) -> C165948
- L1: LCSC (none) -> C1046
Changed lines of the file:
@@
 F 2 "footprints:HRO-TYPE-C-31-M-12-C165948" H 8750 2200 50  0001 C CNN
 F 3 "http://www.usb.org/developers/docs/usb_31_033017.zip" H 8750 2200 50  0001 C CNN
+F 4 "C165948" H 8600 2200 50  0001 C CNN "LCSC"
 	1    8600 2200
 	1    0    0    -1
@@
 F 2 "Inductor_SMD:L_0805_2012Metric" H 4100 3150 50  0001 C CNN
 F 3 "~" H 4100 3150 50  0001 C CNN
+F 4 "C1046" H 4100 3150 50  0001 C CNN "LCSC"
 	1    4100 3150
 	1    0    0    -1

Commit message: fixed bluemacro840 schematic in docs
Connections:
- net labels added: P1.02
- net labels removed: DFU
- no-connect marks 14 -> 13
Changed lines of the file:
@@
 encoding utf-8
 Sheet 1 1
-Title "BlueMacro840"
+Title "BlueMacro840 V2"
 Date ""
 Rev "0.1"
@@
 NoConn ~ 5700 1700
 NoConn ~ 5700 1800
-NoConn ~ 5700 2500
 Text GLabel 6850 1500 2    50   Input ~ 0
 Reset
@@
 Text GLabel 4100 1850 2    50   Input ~ 0
 SWO
-Text GLabel 4100 1650 2    50   Input ~ 0
-DFU
 $Comp
 L Connector_Generic:Conn_01x02 J1
@@
 P0.30
 Text Label 6700 2700 0    50   ~ 0
-P1.06
+P1.02
 Text Label 2200 1650 2    50   ~ 0
 P0.02
@@
 Text Label 2200 2750 2    50   ~ 0
 P0.04
-Text Label 6700 2500 0    50   ~ 0
+Text Label 5700 2500 2    50   ~ 0
 P0.04
 Text Label 2200 2650 2    50   ~ 0
@@
 Text Label 4550 7600 0    50   ~ 0
 P1.00
+Text Label 4100 1650 0    50   ~ 0
+P1.02
+Text Label 6700 2500 0    50   ~ 0
+P1.06
 $EndSCHEMATC
