File: BlueNano/BlueNano 2.0/NRF52832 Base.sch (KiCad schematic (older format))
At the start: 39 parts, among them J1 Conn_01x06, J2 USB_B_Micro, Q1 LP0404N3T5G, U1 NRF52832-QFAA-R, U2 ProMicro, U3 AP2112K-3.3, U4 TP4054ST, U5 CP2104, Y1 32MHz, Y2 32.768kHz

Commit message: fixed bluemacro840 schematic in docs
Parts:
- R1: LCSC (none) -> C29263
- R2: LCSC (none) -> C11512
- U1: LCSC (none) -> C77540
- U5: LCSC (none) -> C47742
Changed lines of the file:
@@
 F 2 "Package_DFN_QFN:QFN-48-1EP_6x6mm_P0.4mm_EP4.66x4.66mm_ThermalVias" H 6450 3740 60  0001 C CNN
 F 3 "" H 4650 3500 60  0000 C CNN
+F 4 "C77540" H 4650 3500 50  0001 C CNN "LCSC"
 	1    4650 3500
 	1    0    0    -1
@@
 F 2 "Resistor_SMD:R_0402_1005Metric" V 4580 1600 50  0001 C CNN
 F 3 "~" H 4650 1600 50  0001 C CNN
+F 4 "C29263" H 4650 1600 50  0001 C CNN "LCSC"
 	1    4650 1600
 	1    0    0    -1
@@
 F 2 "Resistor_SMD:R_0402_1005Metric" V 4580 2050 50  0001 C CNN
 F 3 "~" H 4650 2050 50  0001 C CNN
+F 4 "C11512" H 4650 2050 50  0001 C CNN "LCSC"
 	1    4650 2050
 	1    0    0    -1
@@
 F 2 "Package_DFN_QFN:QFN-24-1EP_4x4mm_P0.5mm_EP2.6x2.6mm" H 10050 750 50  0001 L CNN
 F 3 "https://www.silabs.com/Support%20Documents/TechnicalDocs/cp2104.pdf" H 9350 2950 50  0001 C CNN
+F 4 "C47742" H 9900 1700 50  0001 C CNN "LCSC"
 	1    9900 1700
 	1    0    0    -1
